File: stepper-motor-driver/boost-gate-driver.kicad_sch (KiCad schematic)
At the start: 0 parts

Commit message: gate drivers
Parts:
- added C37: 100nF, symbol Device:C
- added C38, C39: 1uF, symbol Device:C
- added D20: MUR120, symbol Device:D
- added R37: 1kR, symbol Device:R
- added U18: IR2125, IR2125:DIL08, symbol IR2125:IR2125
Connections:
- new net: C38.1, R37.1, U18.3 (ERR)
- new net: C39.1, D20.1 (K), U18.8 (VB)
- new net: C39.2, U18.5 (VS), U18.6 (CS)
- new net +15V: C37.1, D20.2 (A), U18.1 (VCC)
- new net GND: C37.2, C38.2, R37.2, U18.4 (COM)
- new net boost_PWM: U18.2 (IN)
- new net boost_gate: U18.7 (HO)
