File: stepper-motor-driver/gate-drivers.kicad_sch (KiCad schematic)
At the start: 0 parts

Commit message: gate drivers
Parts:
- added C25, C27, C29, C30, C32, C33, C35, C36, C41, C43, C44, C45, C48, C49, C50, C51: 1uF, symbol Device:C
- added C26, C28, C31, C34, C40, C42, C46, C47: 100nF, symbol Device:C
- added D16, D17, D18, D19, D21, D22, D23, D24: MUR120, symbol Device:D
- added R33, R34, R35, R36, R38, R39, R40, R41: 1kR, symbol Device:R
- added U14, U15, U16, U17, U19, U20, U21, U22: IR2125, IR2125:DIL08, symbol IR2125:IR2125
Connections:
- new net: C50.1, D23.1 (K), U21.8 (VB)
- new net: C50.2, U21.5 (VS), U21.6 (CS)
- new net: C51.1, D24.1 (K), U22.8 (VB)
- new net: C51.2, U22.5 (VS), U22.6 (CS)
- new net: C44.1, D21.1 (K), U19.8 (VB)
- new net: C29.1, R36.1, U15.3 (ERR)
- new net: C35.1, R35.1, U17.3 (ERR)
- new net: C25.1, R33.1, U14.3 (ERR)
- new net: C27.2, U14.5 (VS), U14.6 (CS)
- new net: C27.1, D16.1 (K), U14.8 (VB)
- new net: C43.1, R39.1, U20.3 (ERR)
- new net: C48.1, R40.1, U21.3 (ERR)
- new net: C32.1, R34.1, U16.3 (ERR)
- new net: C36.1, D19.1 (K), U17.8 (VB)
- new net: C36.2, U17.5 (VS), U17.6 (CS)
- new net: C49.1, R41.1, U22.3 (ERR)
- new net: C41.1, R38.1, U19.3 (ERR)
- new net: C44.2, U19.5 (VS), U19.6 (CS)
- new net: C30.2, U15.5 (VS), U15.6 (CS)
- new net: C30.1, D17.1 (K), U15.8 (VB)
- new net: C33.1, D18.1 (K), U16.8 (VB)
- new net: C33.2, U16.5 (VS), U16.6 (CS)
- new net: C45.1, D22.1 (K), U20.8 (VB)
- new net: C45.2, U20.5 (VS), U20.6 (CS)
- new net #coil_1: U15.7 (HO), U21.7 (HO)
- new net #coil_2: U17.7 (HO), U22.7 (HO)
- new net #delay_1: U15.2 (IN), U21.2 (IN)
- new net #delay_2: U17.2 (IN), U22.2 (IN)
- new net +15V: C26.1, C28.1, C31.1, C34.1, C40.1, C42.1, C46.1, C47.1, D16.2 (A), D17.2 (A), D18.2 (A), D19.2 (A), D21.2 (A), D22.2 (A), D23.2 (A), D24.2 (A), U14.1 (VCC), U15.1 (VCC), U16.1 (VCC), U17.1 (VCC), U19.1 (VCC), U20.1 (VCC), U21.1 (VCC), U22.1 (VCC)
- new net GND: C25.2, C26.2, C28.2, C29.2, C31.2, C32.2, C34.2, C35.2, C40.2, C41.2, C42.2, C43.2, C46.2, C47.2, C48.2, C49.2, R33.2, R34.2, R35.2, R36.2, R38.2, R39.2, R40.2, R41.2, U14.4 (COM), U15.4 (COM), U16.4 (COM), U17.4 (COM), U19.4 (COM), U20.4 (COM), U21.4 (COM), U22.4 (COM)
- new net coil_1: U14.7 (HO), U20.7 (HO)
- new net coil_2: U16.7 (HO), U19.7 (HO)
- new net delay_1: U14.2 (IN), U20.2 (IN)
- new net delay_2: U16.2 (IN), U19.2 (IN)
