File: motor-driver/h-bridge.kicad_sch (KiCad schematic)
At the start: 24 parts, among them Q1 IRF540N, Q2 IRF540N, Q3 IRF540N, Q4 IRF540N, Q5 IRF540N, Q6 IRF540N, Q7 IRF540N, Q8 IRF540N

Commit message: pcb layout
Parts:
- D10, D11, D12, D5, D6, D7, D8, D9: footprint (none) -> Diode_THT:D_DO-41_SOD81_P12.70mm_Horizontal
Other:
- moved on the sheet: TP12
Changed lines of the file:
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@@
 	)
 	(junction
+		(at 149.86 59.69)
+		(diameter 0)
+		(color 0 0 0 0)
+	)
+	(junction
 		(at 168.91 59.69)
 		(diameter 0)
@@
 	)
 	(junction
-		(at 149.098 59.69)
-		(diameter 0)
-		(color 0 0 0 0)
-	)
-	(junction
 		(at 168.91 105.41)
 		(diameter 0)
@@
 	(wire
 		(pts
-			(xy 149.098 59.69) (xy 153.67 59.69)
-		)
-		(stroke
-			(width 0)
-			(type default)
-		)
-	)
-	(wire
-		(pts
 			(xy 153.67 41.91) (xy 153.67 35.56)
 		)
@@
 	(wire
 		(pts
+			(xy 149.86 59.69) (xy 153.67 59.69)
+		)
+		(stroke
+			(width 0)
+			(type default)
+		)
+	)
+	(wire
+		(pts
 			(xy 82.55 67.31) (xy 87.63 67.31)
 		)
@@
 	(wire
 		(pts
-			(xy 143.51 59.69) (xy 149.098 59.69)
+			(xy 143.51 59.69) (xy 149.86 59.69)
 		)
 		(stroke
@@
 	(wire
 		(pts
-			(xy 149.098 55.88) (xy 149.098 59.69)
+			(xy 149.86 57.15) (xy 149.86 59.69)
 		)
 		(stroke
@@
 			)
 		)
-		(property "Footprint" ""
+		(property "Footprint" "Diode_THT:D_DO-41_SOD81_P12.70mm_Horizontal"
 			(at 110.49 71.12 0)
 			(effects
@@
 			)
 		)
-		(property "Footprint" ""
+		(property "Footprint" "Diode_THT:D_DO-41_SOD81_P12.70mm_Horizontal"
 			(at 153.67 71.12 0)
 			(effects
@@
 	(symbol
 		(lib_id "Connector:TestPoint")
-		(at 149.098 55.88 0)
+		(at 149.86 57.15 0)
 		(mirror y)
 		(unit 1)
@@
 		(fields_autoplaced yes)
 		(property "Reference" "TP12"
-			(at 146.558 51.3079 0)
+			(at 147.32 52.5779 0)
 			(effects
 				(font
@@
 		)
 		(property "Value" "TestPoint"
-			(at 146.558 53.8479 0)
+			(at 147.32 55.1179 0)
 			(effects
 				(font
@@
 		)
 		(property "Footprint" "TestPoint:TestPoint_Loop_D2.50mm_Drill1.0mm"
-			(at 144.018 55.88 0)
+			(at 144.78 57.15 0)
 			(effects
 				(font
@@
 		)
 		(property "Datasheet" "~"
-			(at 144.018 55.88 0)
+			(at 144.78 57.15 0)
 			(effects
 				(font
@@
 		)
 		(property "Description" "test point"
-			(at 149.098 55.88 0)
+			(at 149.86 57.15 0)
 			(effects
 				(font
@@
 			)
 		)
-		(property "Footprint" ""
+		(property "Footprint" "Diode_THT:D_DO-41_SOD81_P12.70mm_Horizontal"
 			(at 153.67 115.57 0)
 			(effects
@@
 			)
 		)
-		(property "Footprint" ""
+		(property "Footprint" "Diode_THT:D_DO-41_SOD81_P12.70mm_Horizontal"
 			(at 153.67 45.72 0)
 			(effects
@@
 			)
 		)
-		(property "Footprint" ""
+		(property "Footprint" "Diode_THT:D_DO-41_SOD81_P12.70mm_Horizontal"
 			(at 153.67 140.97 0)
 			(effects
@@
 			)
 		)
-		(property "Footprint" ""
+		(property "Footprint" "Diode_THT:D_DO-41_SOD81_P12.70mm_Horizontal"
 			(at 110.49 140.97 0)
 			(effects
@@
 			)
 		)
-		(property "Footprint" ""
+		(property "Footprint" "Diode_THT:D_DO-41_SOD81_P12.70mm_Horizontal"
 			(at 110.49 115.57 0)
 			(effects
@@
 			)
 		)
-		(property "Footprint" ""
+		(property "Footprint" "Diode_THT:D_DO-41_SOD81_P12.70mm_Horizontal"
 			(at 110.49 45.72 0)
 			(effects
